Commit message: sdf调试，试图解决相机模型乱跳问题

File: buddi_gazebo/urdf/buddi_devel.urdf (robot description, URDF)
Before this commit: robot buddi, 15 links, 14 joints
Links:
- link base_link: geometry collision mesh filename=/home/hz/hz/Work/Grabotics/B1-project/B1-Simulation/b1_simu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; visual mesh filename=/home/hz/hz/Work/Grabotics/B1-project/B1-Simulation/b1_simu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
- link caster_back_left_link: geometry collision mesh filename=/home/hz/hz/Work/Grabotics/B1-project/B1-Simulation/b1_simu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; visual mesh filename=/home/hz/hz/Work/Grabotics/B1-project/B1-Simulation/b1_simu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
- link caster_back_right_link: geometry collision mesh filename=/home/hz/hz/Work/Grabotics/B1-project/B1-Simulation/b1_simu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; visual mesh filename=/home/hz/hz/Work/Grabotics/B1-project/B1-Simulation/b1_simu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
- link caster_forward_left_link: geometry collision mesh filename=/home/hz/hz/Work/Grabotics/B1-project/B1-Simulation/b1_simu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; visual mesh filename=/home/hz/hz/Work/Grabotics/B1-project/B1-Simulation/b1_simu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
- link caster_forward_right_link: geometry collision mesh filename=/home/hz/hz/Work/Grabotics/B1-project/B1-Simulation/b1_simu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; visual mesh filename=/home/hz/hz/Work/Grabotics/B1-project/B1-Simulation/b1_simu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
- link imu_link: geometry collision mesh filename=/home/hz/hz/Work/Grabotics/B1-project/B1-Simulation/b1_simu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; visual mesh filename=/home/hz/hz/Work/Grabotics/B1-project/B1-Simulation/b1_simu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
- link lidar_back_link: geometry collision mesh filename=/home/hz/hz/Work/Grabotics/B1-project/B1-Simulation/b1_simu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; visual mesh filename=/home/hz/hz/Work/Grabotics/B1-project/B1-Simulation/b1_simu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
- link lidar_forward_link: geometry collision mesh filename=/home/hz/hz/Work/Grabotics/B1-project/B1-Simulation/b1_simu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; visual mesh filename=/home/hz/hz/Work/Grabotics/B1-project/B1-Simulation/b1_simu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
- link rgbd_back_down_link: geometry collision mesh filename=/home/hz/hz/Work/Grabotics/B1-project/B1-Simulation/b1_simu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; visual mesh filename=/home/hz/hz/Work/Grabotics/B1-project/B1-Simulation/b1_simu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
- link rgbd_back_up_link: geometry collision mesh filename=/home/hz/hz/Work/Grabotics/B1-project/B1-Simulation/b1_simu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; visual mesh filename=/home/hz/hz/Work/Grabotics/B1-project/B1-Simulation/b1_simu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
- link rgbd_forward_down_link: geometry collision mesh filename=/home/hz/hz/Work/Grabotics/B1-project/B1-Simulation/b1_simu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; visual mesh filename=/home/hz/hz/Work/Grabotics/B1-project/B1-Simulation/b1_simu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
- link rgbd_forward_up_link: geometry collision mesh filename=/home/hz/hz/Work/Grabotics/B1-project/B1-Simulation/b1_simu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; visual mesh filename=/home/hz/hz/Work/Grabotics/B1-project/B1-Simulation/b1_simu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
- link wheel_left_link: geometry collision mesh filename=/home/hz/hz/Work/Grabotics/B1-project/B1-Simulation/b1_simu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; visual mesh filename=/home/hz/hz/Work/Grabotics/B1-project/B1-Simulation/b1_simu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
- link wheel_right_link: geometry collision mesh filename=/home/hz/hz/Work/Grabotics/B1-project/B1-Simulation/b1_simu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; visual mesh filename=/home/hz/hz/Work/Grabotics/B1-project/B1-Simulation/b1_simu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

Commit message: Fix the bug of sensor config

File: buddi_gazebo/urdf/buddi_devel.urdf (robot description, URDF)
Before this commit: robot buddi, 15 links, 14 joints
Links:
- link base_link: geometry collision mesh filename=/home/hz/hz/Work/Grabotics/b1_simulation/b1-simulation_v2/s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; visual mesh filename=/home/hz/hz/Work/Grabotics/b1_simulation/b1-simulation_v2/s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
- link caster_back_left_link: geometry collision mesh filename=/home/hz/hz/Work/Grabotics/b1_simulation/b1-simulation_v2/s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; visual mesh filename=/home/hz/hz/Work/Grabotics/b1_simulation/b1-simulation_v2/s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
- link caster_back_right_link: geometry collision mesh filename=/home/hz/hz/Work/Grabotics/b1_simulation/b1-simulation_v2/s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; visual mesh filename=/home/hz/hz/Work/Grabotics/b1_simulation/b1-simulation_v2/s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
- link caster_forward_left_link: geometry collision mesh filename=/home/hz/hz/Work/Grabotics/b1_simulation/b1-simulation_v2/s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; visual mesh filename=/home/hz/hz/Work/Grabotics/b1_simulation/b1-simulation_v2/s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
- link caster_forward_right_link: geometry collision mesh filename=/home/hz/hz/Work/Grabotics/b1_simulation/b1-simulation_v2/s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; visual mesh filename=/home/hz/hz/Work/Grabotics/b1_simulation/b1-simulation_v2/s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
- link imu_link: geometry collision mesh filename=/home/hz/hz/Work/Grabotics/b1_simulation/b1-simulation_v2/s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; visual mesh filename=/home/hz/hz/Work/Grabotics/b1_simulation/b1-simulation_v2/s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
- link lidar_back_link: geometry collision mesh filename=/home/hz/hz/Work/Grabotics/b1_simulation/b1-simulation_v2/s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; visual mesh filename=/home/hz/hz/Work/Grabotics/b1_simulation/b1-simulation_v2/s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
- link lidar_forward_link: geometry collision mesh filename=/home/hz/hz/Work/Grabotics/b1_simulation/b1-simulation_v2/s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; visual mesh filename=/home/hz/hz/Work/Grabotics/b1_simulation/b1-simulation_v2/s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
- link rgbd_back_down_link: geometry collision mesh filename=/home/hz/hz/Work/Grabotics/b1_simulation/b1-simulation_v2/s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; visual mesh filename=/home/hz/hz/Work/Grabotics/b1_simulation/b1-simulation_v2/s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
- link rgbd_back_up_link: geometry collision mesh filename=/home/hz/hz/Work/Grabotics/b1_simulation/b1-simulation_v2/s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; visual mesh filename=/home/hz/hz/Work/Grabotics/b1_simulation/b1-simulation_v2/s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
- link rgbd_forward_down_link: geometry collision mesh filename=/home/hz/hz/Work/Grabotics/b1_simulation/b1-simulation_v2/s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; visual mesh filename=/home/hz/hz/Work/Grabotics/b1_simulation/b1-simulation_v2/s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
- link rgbd_forward_up_link: geometry collision mesh filename=/home/hz/hz/Work/Grabotics/b1_simulation/b1-simulation_v2/s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; visual mesh filename=/home/hz/hz/Work/Grabotics/b1_simulation/b1-simulation_v2/s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
- link wheel_left_link: geometry collision mesh filename=/home/hz/hz/Work/Grabotics/b1_simulation/b1-simulation_v2/s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; visual mesh filename=/home/hz/hz/Work/Grabotics/b1_simulation/b1-simulation_v2/s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
- link wheel_right_link: geometry collision mesh filename=/home/hz/hz/Work/Grabotics/b1_simulation/b1-simulation_v2/s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; visual mesh filename=/home/hz/hz/Work/Grabotics/b1_simulation/b1-simulation_v2/s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
